Commit message: Add dual-arm compute_ik/compute_fk for UMI retarget.

File: urdf/lite.urdf (robot description, URDF)
Before this commit: robot lite_000_asm, 24 links, 23 joints
Links:
- added link left_gripper_joint_link, mass 1e-9
- added link right_gripper_joint_link, mass 1e-9
Joints:
- added joint left_gripper_finger_left_joint: type prismatic, parent left_wrist_pitch_link, child left_gripper_finger_left_link, origin xyz=0.1040961904 -0.04585909073 -0.01258790935 rpy=1.5708 -0.0698132 0.845028, axis 1 0 0, limit lower=0 upper=0.047 effort=1 velocity=1, mimic joint=left_gripper multiplier=0.047 offset=0
- added joint right_gripper_finger_left_joint: type prismatic, parent right_wrist_pitch_link, child right_gripper_finger_left_link, origin xyz=0.113421574 -0.009254971529 -0.01265282701 rpy=1.5708 -0.0698132 1.17725, axis 1 0 0, limit lower=0 upper=0.047 effort=1 velocity=1, mimic joint=right_gripper multiplier=0.047 offset=0
- joint left_gripper: child left_gripper_finger_left_link -> left_gripper_joint_link; limit lower=0 upper=0.047 effort=1 velocity=1 -> lower=0 upper=1 effort=1 velocity=1; origin xyz=0.1040961904 -0.04585909073 -0.01258790935 rpy=1.5708 -0.0698132 0.845028 -> xyz=0 0 0 rpy=0 0 0
- joint left_gripper_passive_joint: mimic joint=left_gripper multiplier=1 offset=0 -> joint=left_gripper multiplier=0.047 offset=0
- joint right_gripper: child right_gripper_finger_left_link -> right_gripper_joint_link; limit lower=0 upper=0.047 effort=1 velocity=1 -> lower=0 upper=1 effort=1 velocity=1; origin xyz=0.113421574 -0.009254971529 -0.01265282701 rpy=1.5708 -0.0698132 1.17725 -> xyz=0 0 0 rpy=0 0 0
- joint right_gripper_passive_joint: mimic joint=right_gripper multiplier=1 offset=0 -> joint=right_gripper multiplier=0.047 offset=0

File: urdf/source/lite.urdf.xacro (robot description, xacro)
@@ -13,4 +13,6 @@
     <xacro:arg name="can_interface_right" default="can1"/>
     <xacro:arg name="calibration_file" default=""/>
+    <!-- Per-finger prismatic travel (m); normalized left/right_gripper is [0, 1]. -->
+    <xacro:property name="gripper_finger_travel_m" value="0.047"/>
     <xacro:include filename="lite.ros2_control.xacro"/>
     <link name="right_wrist_yaw_motor_link">
@@ -479,4 +481,18 @@
     </link>
     <link name="right_gripper_tip_middle_link">
+        <inertial>
+            <origin xyz="0 0 0" rpy="0 0 0" />
+            <mass value="1e-9" />
+            <inertia ixx="1e-12" ixy="0" ixz="0" iyy="1e-12" iyz="0" izz="1e-12" />
+        </inertial>
+    </link>
+    <link name="left_gripper_joint_link">
+        <inertial>
+            <origin xyz="0 0 0" rpy="0 0 0" />
+            <mass value="1e-9" />
+            <inertia ixx="1e-12" ixy="0" ixz="0" iyy="1e-12" iyz="0" izz="1e-12" />
+        </inertial>
+    </link>
+    <link name="right_gripper_joint_link">
         <inertial>
             <origin xyz="0 0 0" rpy="0 0 0" />
@@ -655,25 +671,51 @@
     <joint name="left_gripper" type="prismatic">
         <parent link="left_wrist_pitch_link" />
+        <child link="left_gripper_joint_link" />
+        <origin xyz="0 0 0" rpy="0 0 0" />
+        <axis xyz="1 0 0" />
+        <limit lower="0" upper="1" effort="1" velocity="1" />
+        <hardware>
+            <motorType>None</motorType>
+            <motorDirection>1</motorDirection>
+            <armature>0</armature>
+        </hardware>
+    </joint>
+    <joint name="left_gripper_finger_left_joint" type="prismatic">
+        <parent link="left_wrist_pitch_link" />
         <child link="left_gripper_finger_left_link" />
         <origin xyz="0.1040961904 -0.04585909073 -0.01258790935" rpy="1.5708 -0.0698132 0.845028" />
         <axis xyz="1 0 0" />
-        <limit lower="0" upper="0.047" effort="1" velocity="1" />
-        <hardware>
-            <motorType>None</motorType>
-            <motorDirection>1</motorDirection>
-            <armature>0</armature>
-        </hardware>
+        <limit lower="0" upper="${gripper_finger_travel_m}" effort="1" velocity="1" />
+        <hardware>
+            <motorType>None</motorType>
+            <motorDirection>1</motorDirection>
+            <armature>0</armature>
+        </hardware>
+        <mimic joint="left_gripper" multiplier="${gripper_finger_travel_m}" offset="0" />
     </joint>
     <joint name="right_gripper" type="prismatic">
+        <parent link="right_wrist_pitch_link" />
+        <child link="right_gripper_joint_link" />
+        <origin xyz="0 0 0" rpy="0 0 0" />
+        <axis xyz="1 0 0" />
+        <limit lower="0" upper="1" effort="1" velocity="1" />
+        <hardware>
+            <motorType>None</motorType>
+            <motorDirection>1</motorDirection>
+            <armature>0</armature>
+        </hardware>
+    </joint>
+    <joint name="right_gripper_finger_left_joint" type="prismatic">
         <parent link="right_wrist_pitch_link" />
         <child link="right_gripper_finger_left_link" />
         <origin xyz="0.113421574 -0.009254971529 -0.01265282701" rpy="1.5708 -0.0698132 1.17725" />
         <axis xyz="1 0 0" />
-        <limit lower="0" upper="0.047" effort="1" velocity="1" />
-        <hardware>
-            <motorType>None</motorType>
-            <motorDirection>1</motorDirection>
-            <armature>0</armature>
-        </hardware>
+        <limit lower="0" upper="${gripper_finger_travel_m}" effort="1" velocity="1" />
+        <hardware>
+            <motorType>None</motorType>
+            <motorDirection>1</motorDirection>
+            <armature>0</armature>
+        </hardware>
+        <mimic joint="right_gripper" multiplier="${gripper_finger_travel_m}" offset="0" />
     </joint>
     <joint name="left_gripper_passive_joint" type="prismatic">
@@ -688,5 +730,5 @@
             <armature>0</armature>
         </hardware>
-        <mimic joint="left_gripper" multiplier="1" offset="0" />
+        <mimic joint="left_gripper" multiplier="${gripper_finger_travel_m}" offset="0" />
     </joint>
     <joint name="right_gripper_passive_joint" type="prismatic">
@@ -701,5 +743,5 @@
             <armature>0</armature>
         </hardware>
-        <mimic joint="right_gripper" multiplier="1" offset="0" />
+        <mimic joint="right_gripper" multiplier="${gripper_finger_travel_m}" offset="0" />
     </joint>
     <joint name="head_camera_joint" type="fixed">
